File: Hardware/Schimatics/TeleMonitor.brd (EAGLE design)
At the start: 75.9 x 50.8 mm, 11 parts

Commit message: uploaded Sche edits
Parts:
- moved RS-485 2.54 mm to (71.1, 7.62)
Routing:
- net RS-485_A: track 10.2 -> 7.65 mm
- net RS-485_B: track 7.65 -> 10.2 mm
Changed lines of the file:
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@@
 <setting verticaltext="up"/>
 </settings>
-<grid distance="0.05" unitdist="inch" unit="inch" style="lines" multiple="1" display="yes" altdistance="0.025" altunitdist="inch" altunit="inch"/>
+<grid distance="0.1" unitdist="inch" unit="inch" style="lines" multiple="1" display="yes" altdistance="0.025" altunitdist="inch" altunit="inch"/>
 <layers>
 <layer number="1" name="Top" color="4" fill="1" visible="yes" active="yes"/>
@@
 <element name="PLC" library="ArpanMTP1" package="DIL40" value="ATMEGA32" x="38.1" y="30.48"/>
 <element name="POWER" library="ArpanMTP1" package="1X2-3.5MM" value="5MM_TERMINAL_BLOCK-3.5MM" x="40.64" y="10.1346"/>
-<element name="RS-485" library="ArpanMTP1" package="1X2-3.5MM" value="5MM_TERMINAL_BLOCK-3.5MM" x="71.14836875" y="10.15780625" rot="R90"/>
+<element name="RS-485" library="ArpanMTP1" package="1X2-3.5MM" value="5MM_TERMINAL_BLOCK-3.5MM" x="71.14836875" y="7.61780625" rot="R90"/>
 <element name="RS-485_ENABLE" library="jumper" package="JP2" value="" x="48.26" y="7.62" rot="R270"/>
 <element name="RS-485_TRANSLATOR" library="maxim" package="DIL08" value="MAX485" x="59.69" y="8.9154" rot="R270">
@@
 <contactref element="RS-485_TRANSLATOR" pad="6"/>
 <contactref element="RS-485" pad="2"/>
-<wire x1="63.5" y1="7.6454" x2="71.12296875" y2="7.6454" width="0.4064" layer="16"/>
-<wire x1="71.12296875" y1="7.6454" x2="71.12296875" y2="7.61960625" width="0.4064" layer="16"/>
+<wire x1="63.5" y1="7.6454" x2="68.58" y2="7.6454" width="0.4064" layer="16"/>
+<wire x1="68.58" y1="7.6454" x2="68.58" y2="5.08" width="0.4064" layer="16"/>
+<wire x1="68.58" y1="5.08" x2="71.12296875" y2="5.08" width="0.4064" layer="16"/>
+<wire x1="71.12296875" y1="5.08" x2="71.12296875" y2="5.07960625" width="0.4064" layer="16"/>
 </signal>
 <signal name="RS-485_A">
 <contactref element="RS-485" pad="1"/>
 <contactref element="RS-485_TRANSLATOR" pad="7"/>
-<wire x1="63.5" y1="10.1854" x2="71.12" y2="10.1854" width="0.4064" layer="16"/>
-<wire x1="71.12" y1="10.1854" x2="71.12" y2="10.16" width="0.4064" layer="16"/>
-<wire x1="71.12" y1="10.16" x2="71.14836875" y2="10.16" width="0.4064" layer="16"/>
-<wire x1="71.14836875" y1="10.16" x2="71.14836875" y2="12.71980625" width="0.4064" layer="16"/>
+<wire x1="63.5" y1="10.1854" x2="71.14836875" y2="10.1854" width="0.4064" layer="16"/>
+<wire x1="71.14836875" y1="10.1854" x2="71.14836875" y2="10.17980625" width="0.4064" layer="16"/>
 </signal>
 <signal name="RS-485_MODE_SELECT">
